Commit message: next-color_for_gazebo

File: homer/urdf/display.xacro (robot description, xacro)
@@ -9,4 +9,12 @@
             <material name="black"/>
         </visual>
+        <collision>
+            <origin xyz="0.0225 0.0 0.0" rpy="0.0 0.0 0.0"/>
+            <geometry>
+                <box size="0.045 0.09 0.05"/>
+            </geometry>
+        </collision>
+        <xacro:box_inertia m="0.002" l="0.045" w="0.09" h="0.05"
+                           xyz="0.0225 0 0" rpy="0 0 0"/>
     </link>
     <link name="in_display">
@@ -18,4 +26,12 @@
             <material name="green"/>
         </visual>
+        <collision>
+            <origin xyz="0.045 0.0 0.0" rpy="0.0 0.0 0.0"/>
+            <geometry>
+                <box size="0.005 0.07 0.03"/>
+            </geometry>
+        </collision>
+        <xacro:box_inertia m="0.001" l="0.005" w="0.07" h="0.03"
+                           xyz="0.045 0 0" rpy="0 0 0"/>
     </link>
     <joint name="display_body_joint" type="fixed">

File: homer/urdf/homer.xacro (robot description, xacro)
@@ -19,4 +19,12 @@
             <material name="black" />
         </visual>
+        <collision>
+            <origin xyz="0.0 0.0 ${chassi_length/2}" rpy="0.0 0.0 0.0" />
+            <geometry>
+                <cylinder radius="${chassi_radius}" length="${chassi_length}" />
+            </geometry>
+        </collision>
+        <xacro:cylinder_inertia m="1.0" r="${chassi_radius}" h="${chassi_length}"
+                           xyz="0 0 ${chassi_length/2}" rpy="0 0 0"/>
     </link>
     <link name="body">
@@ -28,4 +36,12 @@
             <material name="yellow" />
         </visual>
+        <collision>
+            <origin xyz="0.0 0.0 0.0" rpy="0.0 0.0 0.0" />
+            <geometry>
+                <cylinder radius="${body_radius}" length="${body_length}" />
+            </geometry>
+        </collision>
+        <xacro:cylinder_inertia m="0.5" r="${body_radius}" h="${body_length}"
+                           xyz="0 0 0" rpy="0 0 0"/>
     </link>
     <xacro:macro name="wheel_link" params="prefix ">
@@ -58,4 +74,12 @@
                 </geometry>
             </visual>
+            <collision>
+                <origin xyz="0.0 0.0 0.0" rpy="0.0 0.0 0.0" />
+                <geometry>
+                    <sphere radius="${wheel_radius/2}" />
+                </geometry>
+            </collision>
+            <xacro:sphere_inertia m="0.2" r="${wheel_radius/2}"
+                           xyz="0 0 0" rpy="0 0 0"/>
         </link>
     </xacro:macro>
