Commit message: added cam

File: homer/urdf/camera.xacro (robot description, xacro)
@@ -1,3 +1,74 @@
 <?xml version="1.0"?>
-<robot xmlns:xacro="http://www.ros.org/wiki/xacro" >
+<robot xmlns:xacro="http://www.ros.org/wiki/xacro">
+    <link name="camera">
+        <visual>
+            <geometry>
+                <box size="0.03 0.03 0.03" />
+            </geometry>
+            <material name="white" />
+        </visual>
+        <collision>
+            <geometry>
+                <box size="0.03 0.03 0.03" />
+            </geometry>
+        </collision>
+        <xacro:box_inertia m="0.01" l="0.03" w="0.03" h="0.03"
+            xyz="0 0 0" rpy="0 0 0" />
+    </link>
+    <link name="camera_linse">
+        <visual>
+            <origin xyz="0.0 0.0 0.0" rpy="0.0 ${pi/2} 0.0" />
+            <geometry>
+                <cylinder radius="0.01" length="0.05" />
+            </geometry>
+            <material name="black" />
+        </visual>
+        <collision>
+            <origin xyz="0.0 0.0 0.0" rpy="0.0 ${pi/2} 0.0" />
+            <geometry>
+                <cylinder radius="0.01" length="0.05" />
+            </geometry>
+        </collision>
+        <xacro:cylinder_inertia m="0.005" r="0.01" h="0.05"
+            xyz="0 0 0" rpy="0 ${pi/2} 0" />
+    </link>
+    <link name="homer_cam" />
+    <joint name="cam_body_joint" type="fixed">
+        <parent link="body" />
+        <child link="camera" />
+        <origin xyz="0.1 0.0 0.06" rpy="0.0 0.0 0.0" />
+    </joint>
+    <joint name="linse_cam" type="fixed">
+        <parent link="camera" />
+        <child link="camera_linse" />
+        <origin xyz="0.0 0.0 0.0" rpy="0.0 0.0 0.0" />
+    </joint>
+    <joint name="camera_optical_joint" type="fixed">
+        <parent link="camera_linse" />
+        <child link="homer_cam" />
+        <origin xyz="0.0 0.0 0.0" rpy="0.0 0.0 0.0" />
+    </joint>
+    <gazebo reference="camera">
+        <material>Gazebo/Orange</material>
+        <sensor name="camera" type="camera">
+            <pose> 0 0 0 0 0 0 </pose>
+            <visualize>true</visualize>
+            <update_rate>10</update_rate>
+            <camera>
+                <horizontal_fov>1.089</horizontal_fov>
+                <image>
+                    <format>R8G8B8</format>
+                    <width>640</width>
+                    <height>480</height>
+                </image>
+                <clip>
+                    <near>0.05</near>
+                    <far>8.0</far>
+                </clip>
+            </camera>
+            <plugin name="camera_controller" filename="libgazebo_ros_camera.so">
+                <frame_name>homer_cam</frame_name>
+            </plugin>
+        </sensor>
+    </gazebo>
 </robot>

File: homer/urdf/homer.urdf.xacro (robot description, xacro)
@@ -5,6 +5,6 @@
     <xacro:include filename="joints.xacro"/>
         <xacro:include filename="display.xacro"/>
-<!--    <xacro:include filename="camera.xacro"/>
-        <xacro:include filename="lidar.xacro"/>
+        <xacro:include filename="camera.xacro"/>
+ <!--        <xacro:include filename="lidar.xacro"/>
         <xacro:include filename="gazebo.xacro"/>
 -->

Commit message: added Gazebo Colors

File: homer/urdf/camera.xacro (robot description, xacro)
@@ -51,4 +51,5 @@
     <gazebo reference="camera">
         <material>Gazebo/Orange</material>
+<!--
         <sensor name="camera" type="camera">
             <pose> 0 0 0 0 0 0 </pose>
@@ -70,5 +71,8 @@
                 <frame_name>homer_cam</frame_name>
             </plugin>
-        </sensor>
+        </sensor> -->
+    </gazebo>
+    <gazebo reference="camera_linse">
+        <material>Gazebo/Black</material>
     </gazebo>
 </robot>

File: homer/urdf/display.xacro (robot description, xacro)
@@ -18,4 +18,7 @@
                            xyz="0.0225 0 0" rpy="0 0 0"/>
     </link>
+    <gazebo reference="display">
+        <material>Gazebo/Black</material>
+    </gazebo>
     <link name="in_display">
         <visual>
@@ -35,4 +38,7 @@
                            xyz="0.045 0 0" rpy="0 0 0"/>
     </link>
+    <gazebo reference="in_display">
+        <material>Gazebo/Green</material>
+    </gazebo>
     <joint name="display_body_joint" type="fixed">
         <parent link="body"/>

File: homer/urdf/homer.xacro (robot description, xacro)
@@ -28,4 +28,7 @@
                            xyz="0 0 ${chassi_length/2}" rpy="0 0 0"/>
     </link>
+    <gazebo reference="chassi">
+        <material>Gazebo/Black</material>
+    </gazebo>
     <link name="body">
         <visual>
@@ -45,4 +48,7 @@
                            xyz="0 0 0" rpy="0 0 0"/>
     </link>
+    <gazebo reference="body">
+        <material>Gazebo/Yellow</material>
+    </gazebo>
     <xacro:macro name="wheel_link" params="prefix ">
         <link name="${prefix}_wheel">
@@ -63,4 +69,7 @@
                 xyz="0 0 0" rpy="${pi/2} 0.0 0.0" />
         </link>
+        <gazebo reference="${prefix}_wheel">
+            <material>Gazebo/Blue</material>
+        </gazebo>
     </xacro:macro>
     <xacro:wheel_link prefix="right" />
@@ -83,4 +92,7 @@
                            xyz="0 0 0" rpy="0 0 0"/>
         </link>
+        <gazebo reference="caster_wheel_${prefix}">
+            <material>Gazebo/Grey</material>
+        </gazebo>
     </xacro:macro>
     <xacro:caster_wheel_link prefix="front" />

Commit message: added cam and Lidar for Gazebo

File: homer/urdf/camera.xacro (robot description, xacro)
@@ -51,5 +51,4 @@
     <gazebo reference="camera">
         <material>Gazebo/Orange</material>
-<!--
         <sensor name="camera" type="camera">
             <pose> 0 0 0 0 0 0 </pose>
@@ -71,5 +70,5 @@
                 <frame_name>homer_cam</frame_name>
             </plugin>
-        </sensor> -->
+        </sensor>
     </gazebo>
     <gazebo reference="camera_linse">

File: homer/urdf/homer.urdf.xacro (robot description, xacro)
@@ -6,5 +6,5 @@
         <xacro:include filename="display.xacro"/>
         <xacro:include filename="camera.xacro"/>
- <!--        <xacro:include filename="lidar.xacro"/> -->
+        <xacro:include filename="lidar.xacro"/>
         <xacro:include filename="gazebo.xacro"/>
 </robot>

File: homer/urdf/lidar.xacro (robot description, xacro)
@@ -1,3 +1,57 @@
 <?xml version="1.0"?>
 <robot xmlns:xacro="http://www.ros.org/wiki/xacro" >
+        <!-- LIDAR -->
+        <link name="laser_frame">
+            <visual>
+                <geometry>
+                    <cylinder radius="0.035" length="0.02"/>
+                </geometry>
+                <material name="black"/>
+            </visual>
+            <collision>
+                <geometry>
+                    <cylinder radius="0.035" length="0.02"/>
+                </geometry>
+                <material name="black"/>
+            </collision>
+            <xacro:cylinder_inertia m="0.01" r="0.035" h="0.02"
+                           xyz="0 0 0" rpy="0 0 0"/>
+        </link>
+        <gazebo reference="laser_frame">
+            <material>Gazebo/Black</material>
+        </gazebo>
+        <joint name="laser_joint" type="fixed">
+            <parent link="base_link"/>
+            <child link="laser_frame"/>
+            <origin xyz="0.0 0.0 0.4" rpy="0.0 0.0 -1.57"/>
+        </joint>
+        <gazebo reference="laser_frame">
+            <material>Gazebo/Black</material>
+            <sensor name="laser" type="ray">
+                <pose> 0 0 0 0 0 0 </pose>
+                <visualize>true</visualize>
+                <update_rate>10</update_rate>
+                <ray>
+                    <scan>
+                        <horizontal>
+                            <samples>360</samples>
+                            <resolution>1</resolution>
+                            <min_angle>0.00</min_angle>
+                            <max_angle>3.14</max_angle>
+                        </horizontal>
+                    </scan>
+                    <range>
+                        <min>0.3</min>
+                        <max>6</max>
+                    </range>
+                </ray>
+                <plugin name="laser_controller" filename="libgazebo_ros_ray_sensor.so">
+                    <ros>
+                        <argument>--ros-args --remap ~/out:=scan</argument> <!-- - -ros-args - -remap ~/out:=scan -->
+                    </ros>
+                    <output_type>sensor_msgs/LaserScan</output_type>
+                    <frame_name>laser_frame</frame_name>
+                </plugin>
+            </sensor>
+        </gazebo>
 </robot>
