Commit message: in work

File: homer/urdf/homer_chassi.xacro (robot description, xacro)
@@ -32,7 +32,7 @@
         </visual>
         <collision>
-            <origin xyz="0.0 0.0 0.0" rpy="0.0 0.0 ${PI}"/>
+            <origin xyz="0.0 0.0 0.0" rpy="${PI/2} 0.0 0.0"/>
             <geometry>
-                <mesh filename="package://homer/meshes/wheel.dae" scale="0.5 0.5 0.5"/>
+                <sphere radius="0.033"/>
             </geometry>
         </collision>
@@ -53,7 +53,7 @@
         </visual>
         <collision>
-            <origin xyz="0.0 0.0 0.0" rpy="0.0 0.0 0.0"/>
+            <origin xyz="0.0 0.0 0.0" rpy="${PI/2} 0.0 0.0"/>
             <geometry>
-                <mesh filename="package://homer/meshes/wheel.dae" scale="0.5 0.5 0.5"/>
+                <sphere radius="0.033"/>
             </geometry>
         </collision>
