Commit message: split it

File: homer/urdf/homer.urdf.xacro (robot description, xacro)
@@ -2,104 +2,10 @@
 <robot xmlns:xacro="http://www.ros.org/wiki/xacro" name="homer">
     <xacro:include filename="material.xacro"/>
-    <!-- Macros -->
-    <xacro:property name="chassi_radius" value="0.093"/>
-    <xacro:property name="chassi_length" value="0.045"/>
-    <xacro:property name="body_radius" value="0.11"/>
-    <xacro:property name="body_length" value="0.345"/>
-    <xacro:property name="wheel_radius" value="0.035"/>
-    <xacro:property name="wheel_length" value="0.028"/>
-    <xacro:property name="caster_wheel_radius" value="0.018"/>
-    <!-- Links -->
-    <link name="base_footprint"/>
-    <link name="base_link"/>
-    <link name="chassi">
-        <visual>
-            <origin xyz="0.0 0.0 ${chassi_length/2}" rpy="0.0 0.0 0.0"/>
-            <geometry>
-                <cylinder radius="${chassi_radius}" length="${chassi_length}"/>
-            </geometry>
-            <material name="black"/>
-        </visual>
-    </link>
-    <link name="body">
-        <visual>
-            <origin xyz="0.0 0.0 0.0" rpy="0.0 0.0 0.0"/>
-            <geometry>
-                <cylinder radius="${body_radius}" length="${body_length}"/>
-            </geometry>
-            <material name="yellow"/>
-        </visual>
-    </link>
-    <xacro:macro name="wheel_link" params="prefix ">
-        <link name="${prefix}_wheel">
-            <visual>
-                <origin xyz="0.0 0.0 0.0" rpy="${pi/2} 0.0 0.0"/>
-                <geometry>
-                    <cylinder radius="${wheel_radius}" length="${wheel_length}"/>
-                </geometry>
-                <material name="blue"/>
-            </visual>
-            <collision>
-                <origin xyz="0.0 0.0 0.0" rpy="${pi/2} 0.0 0.0"/>
-                <geometry>
-                    <cylinder radius="${wheel_radius}" length="${wheel_length}"/>
-                </geometry>
-            </collision>
-            <xacro:cylinder_inertia m="0.3" r="${wheel_radius}" h="${wheel_length}"
-                           xyz="0 0 0" rpy="${pi/2} 0.0 0.0"/>
-        </link>
-    </xacro:macro>
-    <xacro:wheel_link prefix="right"/>
-    <xacro:wheel_link prefix="left"/>
-    <xacro:macro name="caster_wheel_link" params="prefix">
-        <link name="caster_wheel_${prefix}">
-            <visual>
-                <origin xyz="0.0 0.0 0.0" rpy="0.0 0.0 0.0"/>
-                <geometry>
-                    <sphere radius="${caster_wheel_radius}"/>
-                </geometry>
-            </visual>
-        </link>
-    </xacro:macro>
-    <xacro:caster_wheel_link prefix="front"/>
-    <xacro:caster_wheel_link prefix="rear"/>
-    <!-- Joints -->
-    <joint name="base_footprint_joint" type="fixed">
-        <parent link="base_footprint"/>
-        <child link="base_link"/>
-        <origin xyz="0.0 0.0 ${wheel_radius}" rpy="0.0 0.0 0.0"/>
-    </joint>
-    <joint name="chassi_joint" type="fixed">
-        <parent link="base_link"/>
-        <child link="chassi"/>
-        <origin xyz="0.0 0.0 0.0" rpy="0.0 0.0 0.0"/>
-    </joint>
-    <joint name="body_joint" type="fixed">
-        <parent link="chassi"/>
-        <child link="body"/>
-        <origin xyz="0.0 0.0 0.21" rpy="0.0 0.0 0.0"/>
-    </joint>
-    <joint name="caster_1" type="fixed">
-        <parent link="chassi"/>
-        <child link="caster_wheel_front"/>
-        <origin xyz="0.085 0.0 -0.016" rpy="0.0 0.0 0.0"/>
-    </joint>
-    <joint name="caster_2" type="fixed">
-        <parent link="chassi"/>
-        <child link="caster_wheel_rear"/>
-        <origin xyz="-0.085 0.0 -0.016" rpy="0.0 0.0 0.0"/>
-    </joint>
-    <!-- Moving Joints-->
-    <joint name="joint_1" type="continuous">
-        <parent link="chassi"/>
-        <child link="right_wheel"/>
-        <axis xyz="0 1 0"/>
-        <origin xyz="0 0.11 0" rpy="0 0 0"/>
-    </joint>
-    <joint name="joint_2" type="continuous">
-        <parent link="chassi"/>
-        <child link="left_wheel"/>
-        <axis xyz="0 1 0"/>
-        <origin xyz="0 -0.11 0" rpy="0 0 0"/>
-    </joint>
+    <xacro:include filename="homer.xacro"/>
+    <xacro:include filename="joints.xacro"/>
+        <xacro:include filename="display.xacro"/>
+<!--    <xacro:include filename="camera.xacro"/>
+        <xacro:include filename="lidar.xacro"/>
+        <xacro:include filename="gazebo.xacro"/>
+-->
 </robot>

Commit message: added ros2_control-- spawner failed at the moment

File: homer/urdf/homer.urdf.xacro (robot description, xacro)
@@ -1,11 +1,11 @@
 <?xml version="1.0"?>
 <robot xmlns:xacro="http://www.ros.org/wiki/xacro" name="homer">
-    <xacro:include filename="material.xacro"/>
-    <xacro:include filename="homer.xacro"/>
-    <xacro:include filename="joints.xacro"/>
-    <xacro:include filename="display.xacro"/>
-    <xacro:include filename="camera.xacro"/>
-    <xacro:include filename="lidar.xacro"/>
-    <xacro:include filename="gazebo.xacro"/>
-   <!-- <xacro:include filename="ros2_control.xacro"/> -->
+    <xacro:include filename="material.xacro" />
+    <xacro:include filename="homer.xacro" />
+    <xacro:include filename="joints.xacro" />
+    <xacro:include filename="display.xacro" />
+    <xacro:include filename="camera.xacro" />
+    <xacro:include filename="lidar.xacro" />
+   <!-- <xacro:include filename="gazebo.xacro"/>  -->
+    <xacro:include filename="ros2_control.xacro" />
 </robot>

File: homer/urdf/homer.xacro (robot description, xacro)
@@ -54,5 +54,5 @@
         <link name="${prefix}_wheel">
             <visual>
-                <origin xyz="0.0 0.0 0.0" rpy="${pi/2} 0.0 0.0" />
+                <origin xyz="0.0 0.0 0.0" rpy="0.0 0.0 0.0" />
                 <geometry>
                     <cylinder radius="${wheel_radius}" length="${wheel_length}" />
@@ -61,11 +61,11 @@
             </visual>
             <collision>
-                <origin xyz="0.0 0.0 0.0" rpy="${pi/2} 0.0 0.0" />
+                <origin xyz="0.0 0.0 0.0" rpy="0.0 0.0 0.0" />
                 <geometry>
-                    <cylinder radius="${wheel_radius}" length="${wheel_length}" />
+                    <sphere radius="${wheel_radius}"/>
                 </geometry>
             </collision>
-            <xacro:cylinder_inertia m="0.3" r="${wheel_radius}" h="${wheel_length}"
-                xyz="0 0 0" rpy="${pi/2} 0.0 0.0" />
+            <xacro:cylinder_inertia m="0.03" r="${wheel_radius}" h="${wheel_length}"
+                xyz="0 0 0" rpy="0.0 0.0 0.0" />
         </link>
         <gazebo reference="${prefix}_wheel">

File: homer/urdf/joints.xacro (robot description, xacro)
@@ -31,12 +31,12 @@
         <parent link="chassi" />
         <child link="right_wheel" />
-        <axis xyz="0 1 0" />
-        <origin xyz="0 0.11 0" rpy="0 0 0" />
+        <axis xyz="0 0 1 " />
+        <origin xyz="0 -0.11 0" rpy="-${pi/2} 0 0" />
     </joint>
     <joint name="joint_2" type="continuous">
         <parent link="chassi" />
         <child link="left_wheel" />
-        <axis xyz="0 1 0" />
-        <origin xyz="0 -0.11 0" rpy="0 0 0" />
+        <axis xyz="0 0 -1" />
+        <origin xyz="0 0.11 0" rpy="${pi/2} 0 0" />
     </joint>
 </robot>

File: homer/urdf/ros2_control.xacro (robot description, xacro)
@@ -7,6 +7,6 @@
         <joint name="joint_1">
             <command_interface name="velocity">
-                <param name="min">-10</param>
-                <param name="max">10</param>
+                <param name="min">-50</param>
+                <param name="max">50</param>
             </command_interface>
             <state_interface name="velocity" />
@@ -15,6 +15,6 @@
         <joint name="joint_2">
             <command_interface name="velocity">
-                <param name="min">-10</param>
-                <param name="max">10</param>
+                <param name="min">-50</param>
+                <param name="max">50</param>
             </command_interface>
             <state_interface name="velocity" />

Commit message: added right files and some tags

File: homer/urdf/homer.urdf.xacro (robot description, xacro)
@@ -1,5 +1,5 @@
 <?xml version="1.0"?>
 <robot xmlns:xacro="http://www.ros.org/wiki/xacro" name="homer">
-    <xacro:include filename="material2.xacro" />
+    <xacro:include filename="material.xacro" />
     <xacro:include filename="homer_chassi.xacro"/>
     <xacro:include filename="homer_body.xacro"/>

File: homer/urdf/homer_body.xacro (robot description, xacro)
@@ -11,4 +11,12 @@
             <material name="yellow" />
         </visual>
+        <collision>
+            <origin xyz="0.0 0.0 0.0" rpy="0.0 0.0 0.0" />
+            <geometry>
+                <mesh filename="package://homer/meshes/LowerCover-Part1.stl"
+                    scale="${scale}" />
+            </geometry>
+        </collision>
+        <xacro:default_inertial mass="1"/>
     </link>
     <joint name="lower_body_1"
@@ -27,4 +35,12 @@
             <material name="yellow" />
         </visual>
+        <collision>
+            <origin xyz="0.0 0.0 0.0" rpy="0.0 0.0 0.0" />
+            <geometry>
+                <mesh filename="package://homer/meshes/LowerCover-Part2.stl"
+                    scale="${scale}" />
+            </geometry>
+        </collision>
+        <xacro:default_inertial mass="1"/>
     </link>
     <joint name="lower_body_2"
@@ -43,4 +59,12 @@
             <material name="yellow" />
         </visual>
+        <collision>
+            <origin xyz="0.0 0.0 0.0" rpy="0.0 0.0 0.0" />
+            <geometry>
+                <mesh filename="package://homer/meshes/LowerCover-Part3.stl"
+                    scale="${scale}" />
+            </geometry>
+        </collision>
+        <xacro:default_inertial mass="1"/>
     </link>
     <joint name="lower_body_3"
@@ -59,4 +83,12 @@
             <material name="yellow" />
         </visual>
+        <collision>
+            <origin xyz="0.0 0.0 0.0" rpy="0.0 0.0 0.0" />
+            <geometry>
+                <mesh filename="package://homer/meshes/LowerCover-Part4.stl"
+                    scale="${scale}" />
+            </geometry>
+        </collision>
+        <xacro:default_inertial mass="1"/>
     </link>
     <joint name="lower_body_4"
@@ -76,4 +108,13 @@
             <material name="black" />
         </visual>
+        <collision>
+            <origin xyz="0.0 0.0 0.0" rpy="0.0 0.0 ${PI}" />
+            <geometry>
+                <mesh
+                    filename="package://homer/meshes/UpperCover-Face-Part1.stl"
+                    scale="${scale}" />
+            </geometry>
+        </collision>
+        <xacro:default_inertial mass="1"/>
     </link>
     <joint name="lower_body_5"
@@ -92,4 +133,12 @@
             <material name="black" />
         </visual>
+        <collision>
+            <origin xyz="0.0 0.0 0.0" rpy="0.0 0.0 0.0" />
+            <geometry>
+                <mesh filename="package://homer/meshes/UpperCover-Part2.stl"
+                    scale="${scale}" />
+            </geometry>
+        </collision>
+        <xacro:default_inertial mass="1"/>
     </link>
     <joint name="lower_body_6"
@@ -108,4 +157,12 @@
             <material name="yellow" />
         </visual>
+        <collision>
+            <origin xyz="0.0 0.0 0.0" rpy="0.0 0.0 0.0" />
+            <geometry>
+                <mesh filename="package://homer/meshes/UpperCover-Part3.stl"
+                    scale="${scale}" />
+            </geometry>
+        </collision>
+        <xacro:default_inertial mass="1"/>
     </link>
     <joint name="lower_body_7"
@@ -124,4 +181,12 @@
             <material name="yellow" />
         </visual>
+        <collision>
+            <origin xyz="0.0 0.0 0.0" rpy="0.0 0.0 0.0" />
+            <geometry>
+                <mesh filename="package://homer/meshes/UpperCover-Part4.stl"
+                    scale="${scale}" />
+            </geometry>
+        </collision>
+        <xacro:default_inertial mass="1"/>
     </link>
     <joint name="lower_body_8"
@@ -141,4 +206,13 @@
             <material name="black" />
         </visual>
+        <collision>
+            <origin xyz="0.0 0.0 0.0" rpy="0.0 ${PI} 0.0" />
+            <geometry>
+                <mesh
+                    filename="package://homer/meshes/LidarTopPlate.stl"
+                    scale="${scale}" />
+            </geometry>
+        </collision>
+        <xacro:default_inertial mass="1"/>
     </link>
     <joint name="lower_body_top"

File: homer/urdf/homer_chassi.xacro (robot description, xacro)
@@ -11,4 +11,11 @@
             <material name="blue"/>
         </visual>
+        <collision>
+            <origin xyz="0.0 0.0 0.0" rpy="0.0 0.0 ${-PI/2}"/>
+            <geometry>
+                <mesh filename="package://homer/meshes/BasePlateHorizontal.stl" scale="${scale}"/>
+            </geometry>
+        </collision>
+        <xacro:default_inertial mass="1"/>
     </link>
     <joint name="virtual_joint" type="fixed">
@@ -24,4 +31,11 @@
             </geometry>
         </visual>
+        <collision>
+            <origin xyz="0.0 0.0 0.0" rpy="0.0 0.0 ${PI}"/>
+            <geometry>
+                <mesh filename="package://homer/meshes/wheel.dae" scale="0.5 0.5 0.5"/>
+            </geometry>
+        </collision>
+        <xacro:default_inertial mass="1"/>
     </link>
     <joint name="joint_1" type="continuous">
@@ -38,4 +52,11 @@
             </geometry>
         </visual>
+        <collision>
+            <origin xyz="0.0 0.0 0.0" rpy="0.0 0.0 0.0"/>
+            <geometry>
+                <mesh filename="package://homer/meshes/wheel.dae" scale="0.5 0.5 0.5"/>
+            </geometry>
+        </collision>
+        <xacro:default_inertial mass="1"/>
     </link>
     <joint name="joint_2" type="continuous">
@@ -52,4 +73,11 @@
             </geometry>
         </visual>
+        <collision>
+            <origin xyz="0.0 0.0 0.0" rpy="0.0 0.0 0.0"/>
+            <geometry>
+                <sphere radius="0.02"/>
+            </geometry>
+        </collision>
+        <xacro:default_inertial mass="1"/>
     </link>
     <joint name="caster_wheel_front" type="fixed">
@@ -65,4 +93,11 @@
             </geometry>
         </visual>
+        <collision>
+            <origin xyz="0.0 0.0 0.0" rpy="0.0 0.0 0.0"/>
+            <geometry>
+                <sphere radius="0.02"/>
+            </geometry>
+        </collision>
+        <xacro:default_inertial mass="1"/>
     </link>
     <joint name="caster_wheel_rear" type="fixed">

File: homer/urdf/material.xacro (robot description, xacro)
@@ -22,4 +22,24 @@
         <color rgba="1 1 0 1"/>
     </material>
+    <xacro:property name="PI" value="3.14159" />
+    <xacro:property name="effort" value="30.0" />
+    <xacro:property name="velocity" value="10.0" />
+    <xacro:macro name="default_inertial" params="mass"> <!-- <xacro:default_inertial mass="1"/> -->
+        <inertial>
+            <mass value="${mass}" />
+            <inertia ixx="1.0" ixy="0.0" ixz="0.0"
+                     iyy="1.0" iyz="0.0"
+                     izz="1.0" />
+        </inertial>
+    </xacro:macro>
+    <xacro:macro name="box_inertia" params="m l w h xyz rpy">
+        <inertial>
+            <origin xyz="${xyz}" rpy="${rpy}" />
+            <mass value="${m}" />
+            <inertia ixx="${(m/12) * (h*h + l*l)}" ixy="0" ixz="0"
+                     iyy="${(m/12) * (w*w + l*l)}" iyz="0"
+                     izz="${(m/12) * (w*w + h*h)}" />
+        </inertial>
+    </xacro:macro>
     <xacro:macro name="box_inertia" params="m l w h xyz rpy">
         <inertial>

Commit message: in work

File: homer/urdf/homer.urdf.xacro (robot description, xacro)
@@ -2,10 +2,10 @@
 <robot xmlns:xacro="http://www.ros.org/wiki/xacro" name="homer">
     <xacro:include filename="material.xacro" />
-    <xacro:include filename="homer_chassi.xacro"/>
+    <xacro:include filename="homer_.xacro"/>
+  <!--   <xacro:include filename="homer_chassi.xacro"/>
     <xacro:include filename="homer_body.xacro"/>
-<!--
     <xacro:include filename="display.xacro" />
-    <xacro:include filename="camera.xacro" /> -->
-    <xacro:include filename="lidar.xacro" />
+    <xacro:include filename="camera.xacro" />
+    <xacro:include filename="lidar.xacro" /> -->
  <!--    <xacro:include filename="gazebo.xacro"/>  -->
     <xacro:include filename="ros2_control.xacro" />

File: homer/urdf/homer_body.xacro (robot description, xacro)
@@ -118,5 +118,5 @@
         <xacro:default_inertial mass="1"/>
     </link>
-    <joint name="lower_body_5"
+    <joint name="upper_body_5"
         type="fixed">
         <parent link="base_link" />
@@ -142,5 +142,5 @@
         <xacro:default_inertial mass="1"/>
     </link>
-    <joint name="lower_body_6"
+    <joint name="upper_body_6"
         type="fixed">
         <parent link="base_link" />
@@ -166,5 +166,5 @@
         <xacro:default_inertial mass="1"/>
     </link>
-    <joint name="lower_body_7"
+    <joint name="upper_body_7"
         type="fixed">
         <parent link="base_link" />
@@ -190,5 +190,5 @@
         <xacro:default_inertial mass="1"/>
     </link>
-    <joint name="lower_body_8"
+    <joint name="upper_body_8"
         type="fixed">
         <parent link="base_link" />
@@ -198,5 +198,5 @@
     <link name="body_top">
         <visual>
-            <origin xyz="0.0 0.0 0.0" rpy="0.0 ${PI} 0.0" />
+            <origin xyz="0.0 0.0 0.0" rpy="0.0 ${PI} ${PI/2}" />
             <geometry>
                 <mesh
@@ -207,5 +207,5 @@
         </visual>
         <collision>
-            <origin xyz="0.0 0.0 0.0" rpy="0.0 ${PI} 0.0" />
+            <origin xyz="0.0 0.0 0.0" rpy="0.0 ${PI} ${PI/2}" />
             <geometry>
                 <mesh
@@ -216,5 +216,5 @@
         <xacro:default_inertial mass="1"/>
     </link>
-    <joint name="lower_body_top"
+    <joint name="body_top_joint"
         type="fixed">
         <parent link="base_link" />

File: homer/urdf/homer_chassi.xacro (robot description, xacro)
@@ -17,5 +17,5 @@
             </geometry>
         </collision>
-        <xacro:default_inertial mass="1"/>
+        <xacro:default_inertial mass="0.3"/>
     </link>
     <joint name="virtual_joint" type="fixed">
@@ -37,5 +37,6 @@
             </geometry>
         </collision>
-        <xacro:default_inertial mass="1"/>
+        <xacro:sphere_inertia m="0.1" r="0.033"
+                           xyz="0 0 0" rpy="${PI/2} 0.0 0.0"/>
     </link>
     <joint name="joint_1" type="continuous">
@@ -58,5 +59,6 @@
             </geometry>
         </collision>
-        <xacro:default_inertial mass="1"/>
+        <xacro:sphere_inertia m="0.1" r="0.033"
+                           xyz="0 0 0" rpy="${PI/2} 0.0 0.0"/>
     </link>
     <joint name="joint_2" type="continuous">
@@ -79,5 +81,6 @@
             </geometry>
         </collision>
-        <xacro:default_inertial mass="1"/>
+        <xacro:sphere_inertia m="0.01" r="0.02"
+                           xyz="0 0 0" rpy="0.0 0.0 0.0"/>
     </link>
     <joint name="caster_wheel_front" type="fixed">
@@ -99,5 +102,6 @@
             </geometry>
         </collision>
-        <xacro:default_inertial mass="1"/>
+        <xacro:sphere_inertia m="0.01" r="0.02"
+                           xyz="0 0 0" rpy="0.0 0.0 0.0"/>
     </link>
     <joint name="caster_wheel_rear" type="fixed">

File: homer/urdf/lidar.xacro (robot description, xacro)
@@ -13,19 +13,16 @@
                     <cylinder radius="0.035" length="0.02"/>
                 </geometry>
-                <material name="black"/>
+                <material name="red"/>
             </collision>
             <xacro:cylinder_inertia m="0.01" r="0.035" h="0.02"
                            xyz="0 0 0" rpy="0 0 0"/>
         </link>
-        <gazebo reference="laser_frame">
-            <material>Gazebo/Black</material>
-        </gazebo>
         <joint name="laser_joint" type="fixed">
-            <parent link="base_link"/>
+            <parent link="body_top"/>
             <child link="laser_frame"/>
-            <origin xyz="0.0 0.0 0.4" rpy="0.0 0.0 -1.57"/>
+            <origin xyz="0.0 0.0 0.01" rpy="0.0 0.0 -1.57"/>
         </joint>
         <gazebo reference="laser_frame">
-            <material>Gazebo/Black</material>
+            <material>Gazebo/Red</material>
             <sensor name="laser" type="ray">
                 <pose> 0 0 0 0 0 0 </pose>

File: homer/urdf/material.xacro (robot description, xacro)
@@ -28,7 +28,7 @@
         <inertial>
             <mass value="${mass}" />
-            <inertia ixx="1.0" ixy="0.0" ixz="0.0"
-                     iyy="1.0" iyz="0.0"
-                     izz="1.0" />
+            <inertia ixx="0.01" ixy="0.0" ixz="0.0"
+                     iyy="0.01" iyz="0.0"
+                     izz="0.01" />
         </inertial>
     </xacro:macro>
