Commit message: ..

File: homer/urdf/material.xacro (robot description, xacro)
@@ -42,13 +42,4 @@
         </inertial>
     </xacro:macro>
-    <xacro:macro name="box_inertia" params="m l w h xyz rpy">
-        <inertial>
-            <origin xyz="${xyz}" rpy="${rpy}" />
-            <mass value="${m}" />
-            <inertia ixx="${(m/12) * (h*h + l*l)}" ixy="0" ixz="0"
-                     iyy="${(m/12) * (w*w + l*l)}" iyz="0"
-                     izz="${(m/12) * (w*w + h*h)}" />
-        </inertial>
-    </xacro:macro>
     <!--
         <xacro:box_inertia m="" l="" w="" h=""
